File: Jam Jar Solar PCB/Jam Jar Solar PCB.sch (KiCad schematic (older format))
At the start: 12 parts, among them J1 SOLAR PV, U1 QX5252

Commit message: Update of PCB and Instructions
Other:
- note removed: "Really want a timer on this?\nRun for 5 hours max?"
Changed lines of the file:
@@
 	1    0    0    -1
 $EndComp
-Text Notes 7900 2100 0    50   ~ 0
-Really want a timer on this?\nRun for 5 hours max?
 $Comp
 L Jam-Jar-Solar-PCB-rescue:LED-Device D4
